File: Electronics/PCB/R107 AC Controller/R107 AC Controller.sch (KiCad schematic (older format))
At the start: 55 parts, among them J1 CAR POWER, J2 CONTROL, J3 ACCESSORY, J4 KNOB, J5 THERMOCOUPLE, J6 USB_B_Mini, J7 ISP, K1 G5LE-1, K2 G5LE-1, Q1 MMBT2222ALT1G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

Commit message: Added PCB README. Changed part for diode D7.
Parts:
- D7: value SS1P3L-M3/84A -> MBR0520LT1G
Changed lines of the file:
@@
 P 9700 4750
 F 0 "D7" H 9700 4967 50  0000 C CNN
-F 1 "SS1P3L-M3/84A" H 9700 4876 50  0000 C CNN
+F 1 "MBR0520LT1G" H 9700 4876 50  0000 C CNN
 F 2 "Britishideas:SMP_DO-220AA" H 9700 4750 50  0001 C CNN
 F 3 "~" H 9700 4750 50  0001 C CNN

Commit message: Updated to current ATmega328P
Parts:
- U1: symbol BritishIdeas:ATmega328P -> R107-AC-Controller-rescue:ATmega328P-BritishIdeas
Changed lines of the file:
@@
 $EndDescr
 $Comp
-L BritishIdeas:ATmega328P U1
+L R107-AC-Controller-rescue:ATmega328P-BritishIdeas U1
 U 1 1 5FE91942
 P 2650 3400
